Commit message: fix some bug

File: descriptions/gx7/urdf/gx7_test.urdf (robot description, URDF)
Before this commit: robot GX7_250721, 8 links, 7 joints
Joints:
- joint joint1: limit lower=-2.0944 upper=2.0944 effort=5 velocity=3.2 -> lower=-3.141592615 upper=3.141592615 effort=5 velocity=3.2
- joint joint2: limit lower=0 upper=3.141592615 effort=5 velocity=3.2 -> lower=-3.141592615 upper=3.141592615 effort=5 velocity=3.2
- joint joint3: limit lower=-2.0944 upper=2.0944 effort=5 velocity=3.2 -> lower=-3.141592615 upper=3.141592615 effort=5 velocity=3.2
- joint joint4: limit lower=0 upper=3.141592615 effort=5 velocity=3.2 -> lower=-3.141592615 upper=3.141592615 effort=5 velocity=3.2
- joint joint5: limit lower=-2.0944 upper=2.0944 effort=5 velocity=3.2 -> lower=-3.141592615 upper=3.141592615 effort=5 velocity=3.2
- joint joint6: limit lower=-1.5707963 upper=1.5707963 effort=5 velocity=3.2 -> lower=-3.141592615 upper=3.141592615 effort=5 velocity=3.2
